File: PCB/PMA-183PLN+/PMA-183PLN+.kicad_sch (KiCad schematic)
At the start: 18 parts, among them J1 Conn_Coaxial, J2 Conn_Coaxial, U1 PMA-183PLN+, U2 MIC5219-2.6YM5-TR

Commit message: pcb: added boms, updated readmes, changed silkscreen from dfs/ems to nmsm
Parts:
- C1, C2, C3, C4, C5, C6, C7, C8: Link (none) -> https://www.digikey.com/en/products/detail/murata-electroni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
- C9: Link (none) -> https://www.digikey.com/en/products/detail/kyocera-avx/TAJA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
- J1, J2: Link (none) -> https://www.digikey.com/en/products/detail/mueller-electric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
- R1, R2: Link (none) -> https://www.digikey.com/en/products/detail/rohm-semiconduct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
- TP1, TP2, TP3: Link (none) -> https://www.digikey.com/en/products/detail/keystone-electro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
- U1: Link (none) -> https://www.minicircuits.com/WebStore/dashboard.html?model=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
- U2: Link (none) -> https://www.digikey.com/en/products/detail/microchip-techno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
Changed lines of the file:
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@@
+      (effects (font (size 1.27 1.27)) hide)
+    )
+    (property "Link" "https://www.digikey.com/en/products/detail/keystone-electronics/5006/255330" (at 81.28 45.72 0)
       (effects (font (size 1.27 1.27)) hide)
     )
@@
     (property "Datasheet" "MIC5219-2.6YM5-TR" (at 125.73 45.72 0)
       (effects (font (size 1.27 1.27) italic) hide)
+    )
+    (property "Link" "https://www.digikey.com/en/products/detail/microchip-technology/MIC5219-2-6YM5-TR/1030548?s=N4IgTCBcDaIKwHYBsBaMC4E4UEYUDkAREAXQF8g" (at 125.73 45.72 0)
+      (effects (font (size 1.27 1.27)) hide)
     )
     (pin "1")
@@
       (effects (font (size 1.27 1.27)) hide)
     )
+    (property "Link" "https://www.digikey.com/en/products/detail/murata-electronics/GRM1555C1H101JA01D/3693829" (at 184.15 95.25 0)
+      (effects (font (size 1.27 1.27)) hide)
+    )
     (pin "1")
     (pin "2")
@@
       (effects (font (size 1.27 1.27)) hide)
     )
+    (property "Link" "https://www.digikey.com/en/products/detail/keystone-electronics/5122/2170325" (at 184.15 45.72 0)
+      (effects (font (size 1.27 1.27)) hide)
+    )
     (pin "1")
     (instances
@@
       (effects (font (size 1.27 1.27)) hide)
     )
+    (property "Link" "https://www.digikey.com/en/products/detail/murata-electronics/GRM1555C1H101JA01D/3693829" (at 119.38 99.06 0)
+      (effects (font (size 1.27 1.27)) hide)
+    )
     (pin "1")
     (pin "2")
@@
     )
     (property "Datasheet" "~" (at 102.87 49.53 0)
+      (effects (font (size 1.27 1.27)) hide)
+    )
+    (property "Link" "https://www.digikey.com/en/products/detail/murata-electronics/GRM155R61H334KE01J/19115579" (at 102.87 49.53 0)
       (effects (font (size 1.27 1.27)) hide)
     )
@@
     )
     (property "Datasheet" "~" (at 158.75 95.25 0)
+      (effects (font (size 1.27 1.27)) hide)
+    )
+    (property "Link" "https://www.digikey.com/en/products/detail/murata-electronics/GRM155R61H334KE01J/19115579" (at 158.75 95.25 0)
       (effects (font (size 1.27 1.27)) hide)
     )
@@
       (effects (font (size 1.27 1.27)) hide)
     )
+    (property "Link" "https://www.digikey.com/en/products/detail/mueller-electric-co/BU-1420761881/11487662" (at 81.28 124.46 0)
+      (effects (font (size 1.27 1.27)) hide)
+    )
     (pin "1")
     (pin "2")
@@
       (effects (font (size 1.27 1.27)) hide)
     )
+    (property "Link" "https://www.digikey.com/en/products/detail/murata-electronics/GRM1555C1H471JA01D/587210" (at 209.55 58.42 0)
+      (effects (font (size 1.27 1.27)) hide)
+    )
     (pin "1")
     (pin "2")
@@
     )
     (property "Datasheet" "~" (at 196.85 58.42 0)
+      (effects (font (size 1.27 1.27)) hide)
+    )
+    (property "Link" "https://www.digikey.com/en/products/detail/kyocera-avx/TAJA225K035RNJ/809523?s=N4IgTCBcDaICwHYAcBaAzABgWlBGFAcgCIgC6AvkA" (at 196.85 58.42 0)
       (effects (font (size 1.27 1.27)) hide)
     )
@@
       (effects (font (size 1.27 1.27)) hide)
     )
+    (property "Link" "https://www.digikey.com/en/products/detail/murata-electronics/GRM155R71H102KA01D/587225" (at 171.45 95.25 0)
+      (effects (font (size 1.27 1.27)) hide)
+    )
     (pin "1")
     (pin "2")
@@
       (effects (font (size 1.27 1.27)) hide)
     )
+    (property "Link" "https://www.digikey.com/en/products/detail/murata-electronics/GRM155R61H334KE01J/19115579" (at 119.38 78.74 0)
+      (effects (font (size 1.27 1.27)) hide)
+    )
     (pin "1")
     (pin "2")
@@
     )
     (property "Datasheet" "~" (at 107.95 45.72 0)
+      (effects (font (size 1.27 1.27)) hide)
+    )
+    (property "Link" "https://www.digikey.com/en/products/detail/keystone-electronics/5005/255329" (at 102.87 45.72 0)
       (effects (font (size 1.27 1.27)) hide)
     )
@@
     (property "Manufacturer_Part_Number" "PMA-183PLN+" (at -633.63 135.89 0)
       (effects (font (size 1.27 1.27)) (justify left top) hide)
+    )
+    (property "Link" "https://www.minicircuits.com/WebStore/dashboard.html?model=PMA-183PLN%2B" (at 151.13 111.76 0)
+      (effects (font (size 1.27 1.27)) hide)
     )
     (pin "1")
@@
       (effects (font (size 1.27 1.27)) hide)
     )
+    (property "Link" "https://www.digikey.com/en/products/detail/rohm-semiconductor/ESR03EZPF1800/4007173" (at 146.05 88.9 0)
+      (effects (font (size 1.27 1.27)) hide)
+    )
     (pin "1")
     (pin "2")
@@
       (effects (font (size 1.27 1.27)) hide)
     )
+    (property "Link" "https://www.digikey.com/en/products/detail/rohm-semiconductor/ESR03EZPF10R0/1983431" (at 184.15 77.47 0)
+      (effects (font (size 1.27 1.27)) hide)
+    )
     (pin "1")
     (pin "2")
@@
     )
     (property "Datasheet" "~" (at 119.38 88.9 0)
+      (effects (font (size 1.27 1.27)) hide)
+    )
+    (property "Link" "https://www.digikey.com/en/products/detail/murata-electronics/GRM155R71H102KA01D/587225" (at 119.38 88.9 0)
       (effects (font (size 1.27 1.27)) hide)
     )
@@
       (effects (font (size 1.27 1.27)) hide)
     )
+    (property "Link" "https://www.digikey.com/en/products/detail/mueller-electric-co/BU-1420761881/11487662" (at 209.55 127 0)
+      (effects (font (size 1.27 1.27)) hide)
+    )
