File: PCB/PMA3-14LN+/PMA3-14LN+.kicad_sch (KiCad schematic)
At the start: 19 parts, among them J1 Conn_Coaxial, J2 Conn_Coaxial, U1 PMA3-14LN+, U2 L7806

Commit message: pcb: added boms, updated readmes, changed silkscreen from dfs/ems to nmsm
Parts:
- C1, C2, C3, C4, C5, C6, C7, C8, C9: Link (none) -> https://www.digikey.com/en/products/detail/murata-electroni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
- J1, J2: Link (none) -> https://www.digikey.com/en/products/detail/mueller-electric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
- L1, L2: Link (none) -> https://www.coilcraft.com/en-us/products/rf/ferrite-core-ch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
- R1: Link (none) -> https://www.digikey.com/en/products/detail/koa-speer-electr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
- TP1, TP2, TP3: Link (none) -> https://www.digikey.com/en/products/detail/keystone-electro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
- U1: Link (none) -> https://www.minicircuits.com/WebStore/dashboard.html?model=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
- U2: Link (none) -> https://www.digikey.com/en/products/detail/stmicroelectroni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
Changed lines of the file:
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@@
+      (effects (font (size 1.27 1.27)) hide)
+    )
+    (property "Link" "https://www.digikey.com/en/products/detail/keystone-electronics/5006/255330" (at 88.9 45.72 0)
       (effects (font (size 1.27 1.27)) hide)
     )
@@
       (effects (font (size 1.27 1.27)) hide)
     )
+    (property "Link" "https://www.digikey.com/en/products/detail/murata-electronics/GRM155R71H103KA88D/1033252" (at 97.79 124.46 0)
+      (effects (font (size 1.27 1.27)) hide)
+    )
     (pin "1")
     (pin "2")
@@
     )
     (property "Datasheet" "~" (at 97.79 101.6 0)
+      (effects (font (size 1.27 1.27)) hide)
+    )
+    (property "Link" "https://www.digikey.com/en/products/detail/murata-electronics/GRM1555C1H101JA01D/3693829" (at 97.79 101.6 0)
       (effects (font (size 1.27 1.27)) hide)
     )
@@
     )
     (property "Datasheet" "~" (at 184.15 130.81 0)
+      (effects (font (size 1.27 1.27)) hide)
+    )
+    (property "Link" "https://www.digikey.com/en/products/detail/murata-electronics/GJM1555C1HR10WB01D/2593239" (at 184.15 130.81 0)
       (effects (font (size 1.27 1.27)) hide)
     )
@@
       (effects (font (size 1.27 1.27)) hide)
     )
+    (property "Link" "https://www.digikey.com/en/products/detail/keystone-electronics/5122/2170325" (at 184.15 45.72 0)
+      (effects (font (size 1.27 1.27)) hide)
+    )
     (pin "1")
     (instances
@@
       (effects (font (size 1.27 1.27)) hide)
     )
+    (property "Link" "https://www.digikey.com/en/products/detail/murata-electronics/GRM1555C1H101JA01D/3693829" (at 194.31 101.6 0)
+      (effects (font (size 1.27 1.27)) hide)
+    )
     (pin "1")
     (pin "2")
@@
       (effects (font (size 1.27 1.27)) hide)
     )
+    (property "Link" "https://www.digikey.com/en/products/detail/murata-electronics/GRM155R61H334KE01J/19115579" (at 121.92 49.53 0)
+      (effects (font (size 1.27 1.27)) hide)
+    )
     (pin "1")
     (pin "2")
@@
     )
     (property "Datasheet" "~" (at 194.31 88.9 0)
+      (effects (font (size 1.27 1.27)) hide)
+    )
+    (property "Link" "https://www.digikey.com/en/products/detail/murata-electronics/GRM155R71H104KE14J/4905180" (at 194.31 88.9 0)
       (effects (font (size 1.27 1.27)) hide)
     )
@@
     )
     (property "Datasheet" "http://www.st.com/content/ccc/resource/technical/document/datasheet/41/4f/b3/b0/12/d4/47/88/CD00000444.pdf/files/CD00000444.pdf/jcr:content/translations/en.CD00000444.pdf" (at 143.51 46.99 0)
+      (effects (font (size 1.27 1.27)) hide)
+    )
+    (property "Link" "https://www.digikey.com/en/products/detail/stmicroelectronics/L7806ABD2T-TR/585696" (at 143.51 45.72 0)
       (effects (font (size 1.27 1.27)) hide)
     )
@@
       (effects (font (size 1.27 1.27)) hide)
     )
+    (property "Link" "https://www.digikey.com/en/products/detail/mueller-electric-co/BU-1420761881/11487662" (at 81.28 124.46 0)
+      (effects (font (size 1.27 1.27)) hide)
+    )
     (pin "1")
     (pin "2")
@@
     )
     (property "Datasheet" "~" (at 107.95 130.81 0)
+      (effects (font (size 1.27 1.27)) hide)
+    )
+    (property "Link" "https://www.digikey.com/en/products/detail/murata-electronics/GJM1555C1HR20WB01D/2593241" (at 107.95 130.81 0)
       (effects (font (size 1.27 1.27)) hide)
     )
@@
     (property "Manufacturer_Part_Number" "PMA3-14LN+" (at 167.64 909.22 0)
       (effects (font (size 1.27 1.27)) (justify left top) hide)
+    )
+    (property "Link" "https://www.minicircuits.com/WebStore/dashboard.html?model=PMA3-14LN%2B" (at 120.65 121.92 0)
+      (effects (font (size 1.27 1.27)) hide)
     )
     (pin "1")
@@
       (effects (font (size 1.27 1.27)) hide)
     )
+    (property "Link" "https://www.coilcraft.com/en-us/products/rf/ferrite-core-chip-inductors/0402-(1005)/0402df/0402df-901/" (at 184.15 113.03 0)
+      (effects (font (size 1.27 1.27)) hide)
+    )
     (pin "1")
     (pin "2")
@@
       (effects (font (size 1.27 1.27)) hide)
     )
+    (property "Link" "https://www.digikey.com/en/products/detail/murata-electronics/GRM155R71H103KA88D/1033252" (at 194.31 124.46 0)
+      (effects (font (size 1.27 1.27)) hide)
+    )
     (pin "1")
     (pin "2")
@@
       (effects (font (size 1.27 1.27)) hide)
     )
+    (property "Link" "https://www.coilcraft.com/en-us/products/rf/ferrite-core-chip-inductors/0402-(1005)/0402df/0402df-901/" (at 107.95 113.03 0)
+      (effects (font (size 1.27 1.27)) hide)
+    )
     (pin "1")
     (pin "2")
@@
       (effects (font (size 1.27 1.27)) hide)
     )
+    (property "Link" "https://www.digikey.com/en/products/detail/keystone-electronics/5005/255329" (at 121.92 45.72 0)
+      (effects (font (size 1.27 1.27)) hide)
+    )
     (pin "1")
     (instances
@@
       (effects (font (size 1.27 1.27)) hide)
     )
+    (property "Link" "https://www.digikey.com/en/products/detail/koa-speer-electronics-inc/RK73H1ETTP5100F/9844229" (at 132.08 88.9 0)
+      (effects (font (size 1.27 1.27)) hide)
+    )
     (pin "1")
     (pin "2")
@@
     )
     (property "Datasheet" "~" (at 97.79 88.9 0)
+      (effects (font (size 1.27 1.27)) hide)
+    )
+    (property "Link" "https://www.digikey.com/en/products/detail/murata-electronics/GRM155R71H104KE14J/4905180" (at 97.79 88.9 0)
       (effects (font (size 1.27 1.27)) hide)
     )
@@
       (effects (font (size 1.27 1.27)) hide)
     )
+    (property "Link" "https://www.digikey.com/en/products/detail/mueller-electric-co/BU-1420761881/11487662" (at 209.55 124.46 0)
+      (effects (font (size 1.27 1.27)) hide)
+    )
