File: PCB/PMA3-14LN+/PMA3-14LN+.kicad_pcb (KiCad board)
At the start: 4 copper layers, 35 x 35 mm, 26 parts, among them J1 Conn_Coaxial, J2 Conn_Coaxial, U1 PMA3-14LN+, U2 L7806

Commit message: Rev C PMA3-14LN+ - Pad Size Change
Routing:
- net GND: vias 168 -> 340
Other:
- board text added: "Remy Nguyen (rev. Natalie Ceonzo)"
- board text added: "Rev C"
- board text removed: "10/24/2024"
- board text removed: "50-10000 MHz SMT LNA"
- board text removed: "B"
- board text removed: "Rev B"
